File: feuchtwerk.kicad_pcb (KiCad board)
At the start: 2 copper layers, 30 x 40 mm, 49 parts, among them P1 CONN_01X04, P2 CONN_01X08, P3 CONN_01X08, U1 STM32F042K6Tx, U2 HDC1080, U3 MCP1754ST-3302E/MB, U4 MCP1754ST-5002E/MB, U5 TJA1051/3, X1 CON_SWD, Y1 8MHz

Commit message: fix wrong light transistor setup, add bmp280 air pressure sensor
Parts:
- removed R3: 220K, Resistors_SMD:R_0603
- removed REF** (x2): Fiducial_1mm_Dia_2.54mm_Outer_CopperTop, Fiducials:Fiducial_1mm_Dia_2.54mm_Outer_CopperTop
- added C13: 100nF, Capacitors_SMD:C_0603, F.Cu at (127.3, 105.6)
- added C14: 100nF, Capacitors_SMD:C_0603, F.Cu at (127.3, 107.1)
- added U6: bmp280, bma280:bmp280, F.Cu at (124.3, 106.4)
- R4: value 220K -> 2K7
- moved X1 5.43 mm to (114.0, 107.2)
- moved R4 2.08 mm to (126.5, 113.5), turned to 0 degrees
- moved R1 2.03 mm to (126.4, 111.2), turned to 180 degrees
Connections:
- R1 pad 1: PHOTO -> +3V3
- R1 pad 2: GND -> PHOTO
Routing:
- net GND: track 162.9 -> 181.4 mm, vias 23 -> 25
- net +3V3: track 165.3 -> 179.1 mm
- net SCL: track 56.5 -> 68.1 mm, vias 4 -> 5
- net SDA: track 52.3 -> 61.1 mm, vias 5 -> 6
- net SWDIO: track 8.25 -> 13.7 mm
- net SWCLK: track 6.43 -> 11.6 mm
- net PHOTO: track 20.6 -> 16.2 mm
- net NRST: track 15.8 -> 17.5 mm
Other:
- outline, holes or cut-outs redrawn
- board text added: "feuchtwerk v1.1"
- board text removed: "feuchtwerk v1.0"
